File: CGA_3_6.sch (KiCad schematic (older format))
At the start: 1 part, among them U4 74S174

Commit message: More sheet 3 drawing
Parts:
- added U1: 74S112, Package_DIP:DIP-16_W7.62mm_LongPads, symbol 74xx:74LS112
- added U26: 74S04, Package_DIP:DIP-14_W7.62mm_LongPads, symbol 74xx:74LS04
- added U42: 74LS86, Package_DIP:DIP-14_W7.62mm_LongPads, symbol 74xx:74LS86
- added U5: 74S174, Package_DIP:DIP-16_W7.62mm_LongPads, symbol 74xx:74LS174
- added U6: 74LS04, Package_DIP:DIP-14_W7.62mm_LongPads, symbol 74xx:74LS04
Connections:
- net labels added: 3.58_MHZ, HCLK, LCLK, Q1, ~14_MHZ, ~7_MHZ, ~HCLK
- wire segments 34 -> 107
- no-connect marks 0 -> 1

Commit message: More sheet 3
Parts:
- added U29: 74S04, Package_DIP:DIP-14_W7.62mm_LongPads, symbol 74xx:74LS04
- added U3: 74S86, Package_DIP:DIP-14_W7.62mm_LongPads, symbol 74xx:74LS86
- added U30: 74LS32, symbol 74xx:74LS32
- added U31: 74LS08, Package_DIP:DIP-14_W7.62mm_LongPads, symbol 74xx:74LS08
- added U49: 74LS02, Package_DIP:DIP-14_W7.62mm_LongPads, symbol 74xx:74LS02
Connections:
- net Q1: now also U3.4
- net Q4: now also U3.13
- net ~LCLK: now also U3.10, U3.2, U3.5
- net at U4.5 (Q1), U4.6 (D2): now also U3.12, U49.2
- net at U5.5 (Q1), U6.11: now also U3.1
- net at U1.9 (Q): now also U3.9
- new net: U29.12, U31.2
- new net: U3.8, U31.1
- new net: U3.3, U30.10
- new net: U30.9, U49.1
- new net CAS_CC: U29.13, U3.11
- new net HRES: U49.3
- new net RAS: U3.6
- new net SL': U30.8
- new net ~CAS: U31.3
Changed lines of the file:
@@
 	2750 1500 3200 1500
 Wire Wire Line
-	3200 1500 3200 700
+	3200 1500 3200 1450
 Wire Wire Line
 	3200 700  1200 700
@@
 Text GLabel 3750 750  2    50   Output ~ 0
 Q4
-Wire Wire Line
-	3250 650  3750 650
-Connection ~ 3250 650
-Text GLabel 3750 650  2    50   Output ~ 0
+Text GLabel 6950 650  2    50   Output ~ 0
 ~LCLK
 $Comp
@@
 U 6 1 61D83074
 P 4550 1650
-F 0 "U6" H 4550 1967 50  0000 C CNN
-F 1 "74LS04" H 4550 1876 50  0000 C CNN
+F 0 "U6" H 4250 1550 50  0000 C CNN
+F 1 "74LS04" H 4750 1550 50  0000 C CNN
 F 2 "Package_DIP:DIP-14_W7.62mm_LongPads" H 4550 1650 50  0001 C CNN
 F 3 "http://www.ti.com/lit/gpn/sn74LS04" H 4550 1650 50  0001 C CNN
@@
 	2750 3600 2950 3600
 Wire Wire Line
-	2950 3600 2950 3100
+	2950 3600 2950 3200
 Wire Wire Line
 	2950 3100 1550 3100
@@
 Wire Wire Line
 	1550 3700 1750 3700
-Wire Wire Line
-	2950 3100 3450 3100
-Connection ~ 2950 3100
-Text GLabel 3450 3100 2    50   Output ~ 0
+Text GLabel 6400 3200 2    50   Output ~ 0
 Q1
 $Comp
@@
 	4250 2150 3050 2150
 Wire Wire Line
-	3050 2150 3050 3700
+	3050 2150 3050 3100
 Wire Wire Line
 	3050 3700 2750 3700
@@
 	3100 1700 3100 1950
 Wire Wire Line
-	3100 1950 5450 1950
+	3100 1950 5150 1950
 Connection ~ 3100 1700
 Wire Wire Line
@@
 Wire Wire Line
 	5650 4150 5650 4950
+Connection ~ 3200 1450
+Wire Wire Line
+	3200 1450 3200 700
+Wire Wire Line
+	5750 1650 5750 1800
+Wire Wire Line
+	5750 1800 5150 1800
+Wire Wire Line
+	5150 1800 5150 1950
+Connection ~ 5150 1950
+Wire Wire Line
+	5150 1950 5450 1950
+Wire Wire Line
+	7450 1550 7550 1550
+Text GLabel 8600 1550 2    50   Output ~ 0
+CAS_CC
+Wire Wire Line
+	3200 1450 6300 1450
+Wire Wire Line
+	5750 1650 6850 1650
+$Comp
+L 74xx:74LS04 U29
+U 6 1 61ED2A1A
+P 8000 1900
+F 0 "U29" H 7950 2100 50  0000 C CNN
+F 1 "74S04" H 7950 1700 50  0000 C CNN
+F 2 "Package_DIP:DIP-14_W7.62mm_LongPads" H 8000 1900 50  0001 C CNN
+F 3 "http://www.ti.com/lit/gpn/sn74LS04" H 8000 1900 50  0001 C CNN
+	6    8000 1900
+	1    0    0    -1
+$EndComp
+$Comp
+L 74xx:74LS86 U?
+U 4 1 61E87976
+P 7150 1550
+AR Path="/60463C10/61E87976" Ref="U?"  Part="4"
+AR Path="/60463C57/61E87976" Ref="U3"  Part="4"
+F 0 "U3" H 7150 1875 50  0000 C CNN
+F 1 "74S86" H 7150 1784 50  0000 C CNN
+F 2 "Package_DIP:DIP-14_W7.62mm_LongPads" H 7150 1550 50  0001 C CNN
+F 3 "74xx/74ls86.pdf" H 7150 1550 50  0001 C CNN
+	4    7150 1550
+	1    0    0    -1
+$EndComp
+Wire Wire Line
+	7550 1550 7550 1900
+Wire Wire Line
+	7550 1900 7700 1900
+Connection ~ 7550 1550
+Wire Wire Line
+	7550 1550 8600 1550
+$Comp
+L 74xx:74LS86 U?
+U 3 1 61EF11FD
+P 7150 2350
+AR Path="/60463C10/61EF11FD" Ref="U?"  Part="4"
+AR Path="/60463C57/61EF11FD" Ref="U3"  Part="3"
+F 0 "U3" H 7150 2050 50  0000 C CNN
+F 1 "74S86" H 7150 2150 50  0000 C CNN
+F 2 "Package_DIP:DIP-14_W7.62mm_LongPads" H 7150 2350 50  0001 C CNN
+F 3 "74xx/74ls86.pdf" H 7150 2350 50  0001 C CNN
+	3    7150 2350
+	1    0    0    1
+$EndComp
+Wire Wire Line
+	3250 650  6600 650
+Connection ~ 3250 650
+Wire Wire Line
+	6850 2250 6700 2250
+Wire Wire Line
+	6600 2250 6600 650
+Connection ~ 6600 650
+Wire Wire Line
+	6600 650  6950 650
+$Comp
+L 74xx:74LS08 U31
+U 1 1 61F27BDC
+P 8750 2000
+F 0 "U31" H 8750 1683 50  0000 C CNN
+F 1 "74LS08" H 8750 1774 50  0000 C CNN
+F 2 "Package_DIP:DIP-14_W7.62mm_LongPads" H 8750 2000 50  0001 C CNN
+F 3 "http://www.ti.com/lit/gpn/sn74LS08" H 8750 2000 50  0001 C CNN
+	1    8750 2000
+	1    0    0    1
+$EndComp
+Wire Wire Line
+	8300 1900 8450 1900
+Wire Wire Line
+	7450 2350 8250 2350
+Wire Wire Line
+	8250 2350 8250 2100
+Wire Wire Line
+	8250 2100 8450 2100
+Wire Wire Line
+	9050 2000 9400 2000
+Text GLabel 9400 2000 2    50   Output ~ 0
+~CAS
+Wire Wire Line
+	6850 2450 6600 2450
+Wire Wire Line
+	6600 2450 6600 4450
+Wire Wire Line
+	6600 4450 6400 4450
+$Comp
+L 74xx:74LS86 U?
+U 2 1 61F435B2
+P 7150 2900
+AR Path="/60463C10/61F435B2" Ref="U?"  Part="4"
+AR Path="/60463C57/61F435B2" Ref="U3"  Part="2"
+F 0 "U3" H 7150 2600 50  0000 C CNN
+F 1 "74S86" H 7150 2700 50  0000 C CNN
+F 2 "Package_DIP:DIP-14_W7.62mm_LongPads" H 7150 2900 50  0001 C CNN
+F 3 "74xx/74ls86.pdf" H 7150 2900 50  0001 C CNN
+	2    7150 2900
+	1    0    0    1
+$EndComp
+Wire Wire Line
+	6700 2250 6700 2800
+Wire Wire Line
+	6700 2800 6850 2800
+Connection ~ 6700 2250
+Wire Wire Line
+	6700 2250 6600 2250
+Wire Wire Line
+	7450 2900 9400 2900
+Text GLabel 9400 2900 2    50   Output ~ 0
+RAS
+Wire Wire Line
+	6850 3000 6200 3000
+Wire Wire Line
+	6200 3000 6200 3200
+Wire Wire Line
+	6200 3200 2950 3200
+Connection ~ 2950 3200
+Wire Wire Line
+	2950 3200 2950 3100
+Wire Wire Line
+	6200 3200 6400 3200
+Connection ~ 6200 3200
+$Comp
+L 74xx:74LS86 U?
+U 1 1 61F94B72
+P 7400 3450
+AR Path="/60463C10/61F94B72" Ref="U?"  Part="4"
+AR Path="/60463C57/61F94B72" Ref="U3"  Part="1"
+F 0 "U3" H 7400 3150 50  0000 C CNN
+F 1 "74S86" H 7400 3250 50  0000 C CNN
+F 2 "Package_DIP:DIP-14_W7.62mm_LongPads" H 7400 3450 50  0001 C CNN
+F 3 "74xx/74ls86.pdf" H 7400 3450 50  0001 C CNN
+	1    7400 3450
+	1    0    0    1
+$EndComp
+Wire Wire Line
+	6700 2800 6700 3350
+Connection ~ 6700 2800
+Wire Wire Line
+	6650 3550 6650 3100
+Wire Wire Line
+	6650 3100 3050 3100
+Connection ~ 3050 3100
+Wire Wire Line
+	3050 3100 3050 3700
+$Comp
+L 74xx:74LS02 U49
+U 1 1 61FB1970
+P 7400 4050
+F 0 "U49" H 7400 4375 50  0000 C CNN
+F 1 "74LS02" H 7400 4284 50  0000 C CNN
+F 2 "Package_DIP:DIP-14_W7.62mm_LongPads" H 7400 4050 50  0001 C CNN
+F 3 "http://www.ti.com/lit/gpn/sn74ls02" H 7400 4050 50  0001 C CNN
+	1    7400 4050
+	1    0    0    -1
+$EndComp
+$Comp
+L 74xx:74LS32 U30
+U 3 1 61FB51C0
+P 8250 3750
+F 0 "U30" H 8250 3433 50  0000 C CNN
+F 1 "74LS32" H 8250 3524 50  0000 C CNN
+F 2 "" H 8250 3750 50  0001 C CNN
+F 3 "http://www.ti.com/lit/gpn/sn74LS32" H 8250 3750 50  0001 C CNN
+	3    8250 3750
+	1    0    0    1
+$EndComp
+Wire Wire Line
+	7700 3450 7800 3450
+Wire Wire Line
+	7800 3450 7800 3650
+Wire Wire Line
+	7800 3650 7950 3650
+Wire Wire Line
+	7700 4050 7800 4050
+Wire Wire Line
+	7800 4050 7800 3850
+Wire Wire Line
+	7800 3850 7950 3850
+Wire Wire Line
+	6300 3950 6300 1450
+Connection ~ 6300 1450
+Wire Wire Line
+	6300 1450 6850 1450
+Text GLabel 6900 4150 0    50   Input ~ 0
+HRES
+Wire Wire Line
+	6700 3350 7100 3350
+Wire Wire Line
+	6650 3550 7100 3550
+Wire Wire Line
+	6300 3950 7100 3950
+Wire Wire Line
+	6900 4150 7100 4150
+Wire Wire Line
+	8550 3750 9400 3750
+Text GLabel 9400 3750 2    50   Output ~ 0
+SL'
 $EndSCHEMATC

Commit message: More sheet 3
Parts:
- added U12: 74LS393, Package_DIP:DIP-14_W7.62mm_LongPads, symbol 74xx:74LS393
- added U65: 74LS02, Package_DIP:DIP-14_W7.62mm_LongPads, symbol 74xx:74LS02
Connections:
- new net: U12.12 (MR), U12.2 (MR), U65.13
- new net V_SYNC_DLY: U12.1 (CP)
- new net ~BLINK: U12.11 (Q0)
- new net ~CURSOR_BLINK: U12.13 (CP), U12.6 (Q3)
- new net ~RESET': U65.11, U65.12
- no-connect marks 1 -> 7
Changed lines of the file:
@@
 Text GLabel 9400 3750 2    50   Output ~ 0
 SL'
+$Comp
+L 74xx:74LS02 U65
+U 4 1 6205C9B5
+P 3850 5800
+F 0 "U65" H 3850 6125 50  0000 C CNN
+F 1 "74LS02" H 3850 6034 50  0000 C CNN
+F 2 "Package_DIP:DIP-14_W7.62mm_LongPads" H 3850 5800 50  0001 C CNN
+F 3 "http://www.ti.com/lit/gpn/sn74ls02" H 3850 5800 50  0001 C CNN
+	4    3850 5800
+	1    0    0    -1
+$EndComp
+Wire Wire Line
+	3550 5900 3400 5900
+Wire Wire Line
+	3400 5900 3400 5700
+Wire Wire Line
+	3400 5700 3550 5700
+Wire Wire Line
+	3400 5700 1300 5700
+Connection ~ 3400 5700
+Text GLabel 1300 5700 0    50   Input ~ 0
+~RESET'
+$Comp
+L 74xx:74LS393 U12
+U 1 1 62072115
+P 5450 5600
+F 0 "U12" H 5450 5967 50  0000 C CNN
+F 1 "74LS393" H 5450 5876 50  0000 C CNN
+F 2 "Package_DIP:DIP-14_W7.62mm_LongPads" H 5450 5600 50  0001 C CNN
+F 3 "74xx\\74LS393.pdf" H 5450 5600 50  0001 C CNN
+	1    5450 5600
+	1    0    0    -1
+$EndComp
+$Comp
+L 74xx:74LS393 U12
+U 2 1 62073AB5
+P 5450 6400
+F 0 "U12" H 5450 6767 50  0000 C CNN
+F 1 "74LS393" H 5450 6676 50  0000 C CNN
+F 2 "Package_DIP:DIP-14_W7.62mm_LongPads" H 5450 6400 50  0001 C CNN
+F 3 "74xx\\74LS393.pdf" H 5450 6400 50  0001 C CNN
+	2    5450 6400
+	1    0    0    -1
+$EndComp
+NoConn ~ 5950 5700
+NoConn ~ 5950 5600
+NoConn ~ 5950 5500
+NoConn ~ 5950 6400
+NoConn ~ 5950 6500
+NoConn ~ 5950 6600
+Wire Wire Line
+	4600 6600 4950 6600
+Wire Wire Line
+	4950 5800 4600 5800
+Wire Wire Line
+	4600 5800 4600 6600
+Wire Wire Line
+	5950 5800 6200 5800
+Wire Wire Line
+	6200 5800 6200 5950
+Wire Wire Line
+	6200 5950 4800 5950
+Wire Wire Line
+	4800 5950 4800 6300
+Wire Wire Line
+	4800 6300 4950 6300
+Wire Wire Line
+	4150 5800 4600 5800
+Connection ~ 4600 5800
+Text GLabel 4650 5500 0    50   Input ~ 0
+V_SYNC_DLY
+Wire Wire Line
+	4650 5500 4950 5500
+Wire Wire Line
+	6200 5800 7050 5800
+Connection ~ 6200 5800
+Text GLabel 7050 5800 2    50   Output ~ 0
+~CURSOR_BLINK
+Wire Wire Line
+	5950 6300 7050 6300
+Text GLabel 7050 6300 2    50   Output ~ 0
+~BLINK
 $EndSCHEMATC

Commit message: More sheet 3
Parts:
- added U15: 74LS00, Package_DIP:DIP-14_W7.62mm_LongPads, symbol 74xx:74LS00
- added U18, U19: 74LS138, Package_DIP:DIP-16_W7.62mm_LongPads, symbol 74xx:74LS138
- added U41: 74LS08, Package_DIP:DIP-14_W7.62mm_LongPads, symbol 74xx:74LS08
- U31: value 74LS08 -> 74S08
Connections:
- net GND: now also U18.8 (GND), U19.8 (GND)
- net VCC: now also U18.16 (VCC), U19.16 (VCC)
- new net: U18.6 (E3), U41.3
- new net: U19.5 (E2), U41.11
- new net A15: U19.1 (A0)
- new net A16: U19.2 (A1)
- new net A17: U19.3 (A2)
- new net A18: U19.4 (E1)
- new net A19: U19.6 (E3)
- new net A4: U18.1 (A0)
- new net A5: U18.5 (E2)
- new net A6: U18.2 (A1)
- new net A7: U18.3 (A2)
- new net A8: U41.2
- new net A9: U41.1
- new net AEN: U18.4 (E1)
- new net CPU_MEM_SEL: U19.7 (O7)
- new net ~IOR: U15.12
- new net ~IOW: U15.13
- new net ~MEMR: U41.12
- new net ~MEMW: U41.13
- no-connect marks 7 -> 21
Changed lines of the file:
@@
 P 8750 2000
 F 0 "U31" H 8750 1683 50  0000 C CNN
-F 1 "74LS08" H 8750 1774 50  0000 C CNN
+F 1 "74S08" H 8750 1774 50  0000 C CNN
 F 2 "Package_DIP:DIP-14_W7.62mm_LongPads" H 8750 2000 50  0001 C CNN
 F 3 "http://www.ti.com/lit/gpn/sn74LS08" H 8750 2000 50  0001 C CNN
@@
 Text GLabel 7050 6300 2    50   Output ~ 0
 ~BLINK
+$Comp
+L 74xx:74LS08 U41
+U 1 1 6213A459
+P 1750 7350
+F 0 "U41" H 2000 7250 50  0000 C CNN
+F 1 "74LS08" H 2050 7400 50  0000 C CNN
+F 2 "Package_DIP:DIP-14_W7.62mm_LongPads" H 1750 7350 50  0001 C CNN
+F 3 "http://www.ti.com/lit/gpn/sn74LS08" H 1750 7350 50  0001 C CNN
+	1    1750 7350
+	1    0    0    1
+$EndComp
+Text GLabel 1150 7250 0    50   Input ~ 0
+A8
+Text GLabel 1150 7450 0    50   Input ~ 0
+A9
+Wire Wire Line
+	1150 7250 1450 7250
+Wire Wire Line
+	1150 7450 1450 7450
+$Comp
+L 74xx:74LS138 U18
+U 1 1 62176A88
+P 3500 7150
+F 0 "U18" H 3250 7600 50  0000 C CNN
+F 1 "74LS138" H 3700 7600 50  0000 C CNN
+F 2 "Package_DIP:DIP-16_W7.62mm_LongPads" H 3500 7150 50  0001 C CNN
+F 3 "http://www.ti.com/lit/gpn/sn74LS138" H 3500 7150 50  0001 C CNN
+	1    3500 7150
+	1    0    0    -1
+$EndComp
+$Comp
+L power:VCC #PWR?
+U 1 1 62178652
+P 3500 6550
+F 0 "#PWR?" H 3500 6400 50  0001 C CNN
+F 1 "VCC" H 3515 6723 50  0000 C CNN
+F 2 "" H 3500 6550 50  0001 C CNN
+F 3 "" H 3500 6550 50  0001 C CNN
+	1    3500 6550
+	1    0    0    -1
+$EndComp
+$Comp
+L power:GND #PWR?
+U 1 1 62178E32
+P 3500 7850
+F 0 "#PWR?" H 3500 7600 50  0001 C CNN
+F 1 "GND" H 3505 7677 50  0000 C CNN
+F 2 "" H 3500 7850 50  0001 C CNN
+F 3 "" H 3500 7850 50  0001 C CNN
+	1    3500 7850
+	1    0    0    -1
+$EndComp
+NoConn ~ 4000 7450
+NoConn ~ 4000 7350
+NoConn ~ 4000 7250
+NoConn ~ 4000 7150
+NoConn ~ 4000 7050
+NoConn ~ 4000 6950
+NoConn ~ 4000 6850
+Wire Wire Line
+	2050 7350 3000 7350
+Text GLabel 1150 7750 0    50   Input ~ 0
+AEN
+Wire Wire Line
+	3000 7550 2900 7550
+Wire Wire Line
+	2900 7550 2900 7750
+Wire Wire Line
+	2900 7750 1150 7750
+Wire Wire Line
+	3000 7450 2800 7450
+Wire Wire Line
+	2800 7450 2800 7600
+Wire Wire Line
+	2800 7600 1150 7600
+Text GLabel 1150 7600 0    50   Input ~ 0
+A5
+Wire Wire Line
+	3000 7050 1150 7050
+Text GLabel 1150 7050 0    50   Input ~ 0
+A7
+Wire Wire Line
+	3000 6950 1150 6950
+Text GLabel 1150 6950 0    50   Input ~ 0
+A6
+Wire Wire Line
+	3000 6850 1150 6850
+Text GLabel 1150 6850 0    50   Input ~ 0
+A4
+$Comp
+L 74xx:74LS138 U19
+U 1 1 62233584
+P 3500 8950
+F 0 "U19" H 3250 9400 50  0000 C CNN
+F 1 "74LS138" H 3700 9400 50  0000 C CNN
+F 2 "Package_DIP:DIP-16_W7.62mm_LongPads" H 3500 8950 50  0001 C CNN
+F 3 "http://www.ti.com/lit/gpn/sn74LS138" H 3500 8950 50  0001 C CNN
+	1    3500 8950
+	1    0    0    -1
+$EndComp
+$Comp
+L power:VCC #PWR?
+U 1 1 62233746
+P 3500 8350
+F 0 "#PWR?" H 3500 8200 50  0001 C CNN
+F 1 "VCC" H 3515 8523 50  0000 C CNN
+F 2 "" H 3500 8350 50  0001 C CNN
+F 3 "" H 3500 8350 50  0001 C CNN
+	1    3500 8350
+	1    0    0    -1
+$EndComp
+$Comp
+L power:GND #PWR?
+U 1 1 62233750
+P 3500 9650
+F 0 "#PWR?" H 3500 9400 50  0001 C CNN
+F 1 "GND" H 3505 9477 50  0000 C CNN
+F 2 "" H 3500 9650 50  0001 C CNN
+F 3 "" H 3500 9650 50  0001 C CNN
+	1    3500 9650
+	1    0    0    -1
+$EndComp
+NoConn ~ 4000 8650
+NoConn ~ 4000 8750
+NoConn ~ 4000 8850
+NoConn ~ 4000 8950
+NoConn ~ 4000 9050
+NoConn ~ 4000 9150
+NoConn ~ 4000 9250
+$Comp
+L 74xx:74LS08 U41
+U 4 1 62283BF0
+P 1750 9250
+F 0 "U41" H 2050 9350 50  0000 C CNN
+F 1 "74LS08" H 2100 9200 50  0000 C CNN
+F 2 "Package_DIP:DIP-14_W7.62mm_LongPads" H 1750 9250 50  0001 C CNN
+F 3 "http://www.ti.com/lit/gpn/sn74LS08" H 1750 9250 50  0001 C CNN
+	4    1750 9250
+	1    0    0    -1
+$EndComp
+Wire Wire Line
+	2050 9250 3000 9250
+Wire Wire Line
+	1450 9150 1100 9150
+Wire Wire Line
+	1450 9350 1100 9350
+Text GLabel 1100 9150 0    50   Input ~ 0
+~MEMR
+Text GLabel 1100 9350 0    50   Input ~ 0
+~MEMW
+Wire Wire Line
+	3000 9350 2400 9350
+Wire Wire Line
+	2400 9350 2400 9550
+Wire Wire Line
+	2400 9550 1100 9550
+Text GLabel 1100 9550 0    50   Input ~ 0
+A18
+Wire Wire Line
+	3000 9150 2400 9150
+Wire Wire Line
+	2400 9150 2400 9000
+Wire Wire Line
+	2400 9000 1100 9000
+Text GLabel 1100 9000 0    50   Input ~ 0
+A19
+Wire Wire Line
+	3000 8850 1100 8850
+Text GLabel 1100 8850 0    50   Input ~ 0
+A17
+Wire Wire Line
+	3000 8750 1100 8750
+Text GLabel 1100 8750 0    50   Input ~ 0
+A16
+Wire Wire Line
+	3000 8650 1100 8650
+Text GLabel 1100 8650 0    50   Input ~ 0
+A15
+$Comp
+L 74xx:74LS00 U15
+U 4 1 6230EF83
+P 1750 10050
+F 0 "U15" H 1750 10375 50  0000 C CNN
+F 1 "74LS00" H 1750 10284 50  0000 C CNN
+F 2 "Package_DIP:DIP-14_W7.62mm_LongPads" H 1750 10050 50  0001 C CNN
+F 3 "http://www.ti.com/lit/gpn/sn74ls00" H 1750 10050 50  0001 C CNN
+	4    1750 10050
+	1    0    0    -1
+$EndComp
+Wire Wire Line
+	1450 9950 1100 9950
+Wire Wire Line
+	1450 10150 1100 10150
+Text GLabel 1100 9950 0    50   Input ~ 0
+~IOR
+Text GLabel 1100 10150 0    50   Input ~ 0
+~IOW
+Text GLabel 4400 9350 2    50   Output ~ 0
+CPU_MEM_SEL
+Wire Wire Line
+	4000 9350 4400 9350
 $EndSCHEMATC

Commit message: More sheet 3
Parts:
- added unit 1 of U30
- added unit 1 of U65
Connections:
- net at U18.7 (O7): now also U30.2, U65.2
- net CPU_MEM_SEL renamed ~CPU_MEM_SEL
- new net A3: U30.1
- new net ~6845_CS: U30.3
Changed lines of the file:
@@
 ~IOW
 Text GLabel 4400 9350 2    50   Output ~ 0
-CPU_MEM_SEL
+~CPU_MEM_SEL
 Wire Wire Line
 	4000 9350 4400 9350
+$Comp
+L 74xx:74LS32 U30
+U 1 1 62367D86
+P 5250 7450
+F 0 "U30" H 5250 7650 50  0000 C CNN
+F 1 "74LS32" H 5250 7750 50  0000 C CNN
+F 2 "" H 5250 7450 50  0001 C CNN
+F 3 "http://www.ti.com/lit/gpn/sn74LS32" H 5250 7450 50  0001 C CNN
+	1    5250 7450
+	1    0    0    -1
+$EndComp
+Wire Wire Line
+	4950 7350 4650 7350
+Text GLabel 4650 7350 0    50   Input ~ 0
+A3
+Wire Wire Line
+	4000 7550 4750 7550
+Wire Wire Line
+	5550 7450 6350 7450
+Text GLabel 6350 7450 2    50   Output ~ 0
+~6845_CS
+$Comp
+L 74xx:74LS02 U65
+U 1 1 623F400E
+P 5250 8050
+F 0 "U65" H 5250 8375 50  0000 C CNN
+F 1 "74LS02" H 5250 8284 50  0000 C CNN
+F 2 "Package_DIP:DIP-14_W7.62mm_LongPads" H 5250 8050 50  0001 C CNN
+F 3 "http://www.ti.com/lit/gpn/sn74ls02" H 5250 8050 50  0001 C CNN
+	1    5250 8050
+	1    0    0    -1
+$EndComp
+Wire Wire Line
+	4750 7550 4750 7950
+Wire Wire Line
+	4750 7950 4950 7950
+Connection ~ 4750 7550
+Wire Wire Line
+	4750 7550 4950 7550
 $EndSCHEMATC

Commit message: More sheet 3
Parts:
- added U11: 74LS74, Package_DIP:DIP-14_W7.62mm_LongPads, symbol 74xx:74LS74
- added U13: 74LS08, Package_DIP:DIP-14_W7.62mm_LongPads, symbol 74xx:74LS08
- added U16: 74LS04, Package_DIP:DIP-14_W7.62mm_LongPads, symbol 74xx:74LS04
- added unit 5 of U29
Connections:
- net VCC: now also U11.10 (~S)
- net ~CPU_MEM_SEL: now also U13.10
- net at U15.11: now also U11.12 (D), U11.13 (~R), U16.1
- net at U65.1: now also U29.11
- net at U65.3: now also U16.2
- new net: U13.9, U29.10
- new net DATA_GATE: U13.8
- new net E: U11.9 (Q)
- new net IO_CLOCK: U11.11 (C)
- no-connect marks 21 -> 22
Other:
- moved on the sheet: U15D
Changed lines of the file:
@@
 L 74xx:74LS00 U15
 U 4 1 6230EF83
-P 1750 10050
-F 0 "U15" H 1750 10375 50  0000 C CNN
-F 1 "74LS00" H 1750 10284 50  0000 C CNN
-F 2 "Package_DIP:DIP-14_W7.62mm_LongPads" H 1750 10050 50  0001 C CNN
-F 3 "http://www.ti.com/lit/gpn/sn74ls00" H 1750 10050 50  0001 C CNN
-	4    1750 10050
+P 5000 8750
+F 0 "U15" H 5000 9075 50  0000 C CNN
+F 1 "74LS00" H 5000 8984 50  0000 C CNN
+F 2 "Package_DIP:DIP-14_W7.62mm_LongPads" H 5000 8750 50  0001 C CNN
+F 3 "http://www.ti.com/lit/gpn/sn74ls00" H 5000 8750 50  0001 C CNN
+	4    5000 8750
 	1    0    0    -1
 $EndComp
 Wire Wire Line
-	1450 9950 1100 9950
+	4700 8650 4350 8650
 Wire Wire Line
-	1450 10150 1100 10150
-Text GLabel 1100 9950 0    50   Input ~ 0
+	4700 8850 4350 8850
+Text GLabel 4350 8650 0    50   Input ~ 0
 ~IOR
-Text GLabel 1100 10150 0    50   Input ~ 0
+Text GLabel 4350 8850 0    50   Input ~ 0
 ~IOW
 Text GLabel 4400 9350 2    50   Output ~ 0
 ~CPU_MEM_SEL
 Wire Wire Line
-	4000 9350 4400 9350
+	4000 9350 4300 9350
 $Comp
 L 74xx:74LS32 U30
@@
 Wire Wire Line
 	4750 7550 4950 7550
+$Comp
+L 74xx:74LS04 U16
+U 1 1 6240B59C
+P 5800 8750
+F 0 "U16" H 5750 8950 50  0000 C CNN
+F 1 "74LS04" H 5750 8550 50  0000 C CNN
+F 2 "Package_DIP:DIP-14_W7.62mm_LongPads" H 5800 8750 50  0001 C CNN
+F 3 "http://www.ti.com/lit/gpn/sn74LS04" H 5800 8750 50  0001 C CNN
+	1    5800 8750
+	1    0    0    -1
+$EndComp
+Wire Wire Line
+	5300 8750 5400 8750
+Wire Wire Line
+	4950 8150 4650 8150
+Wire Wire Line
+	4650 8150 4650 8300
+Wire Wire Line
+	4650 8300 6350 8300
+Wire Wire Line
+	6350 8300 6350 8750
+Wire Wire Line
+	6350 8750 6100 8750
+$Comp
+L 74xx:74LS04 U29
+U 5 1 6245A7B3
+P 6150 8050
+F 0 "U29" H 6100 8250 50  0000 C CNN
+F 1 "74S04" H 6100 7850 50  0000 C CNN
+F 2 "Package_DIP:DIP-14_W7.62mm_LongPads" H 6150 8050 50  0001 C CNN
+F 3 "http://www.ti.com/lit/gpn/sn74LS04" H 6150 8050 50  0001 C CNN
+	5    6150 8050
+	1    0    0    -1
+$EndComp
+Wire Wire Line
+	5550 8050 5850 8050
+$Comp
+L 74xx:74LS08 U13
+U 3 1 62471307
+P 7000 8150
+F 0 "U13" H 7300 8250 50  0000 C CNN
+F 1 "74LS08" H 7350 8100 50  0000 C CNN
+F 2 "Package_DIP:DIP-14_W7.62mm_LongPads" H 7000 8150 50  0001 C CNN
+F 3 "http://www.ti.com/lit/gpn/sn74LS08" H 7000 8150 50  0001 C CNN
+	3    7000 8150
+	1    0    0    -1
+$EndComp
+Wire Wire Line
+	6450 8050 6700 8050
+Wire Wire Line
+	4300 9350 4300 9100
+Wire Wire Line
+	4300 9100 6500 9100
+Wire Wire Line
+	6500 9100 6500 8250
+Wire Wire Line
+	6500 8250 6700 8250
+Connection ~ 4300 9350
+Wire Wire Line
+	4300 9350 4400 9350
+Text GLabel 7700 8150 2    50   Output ~ 0
+DATA_GATE
+Wire Wire Line
+	7300 8150 7700 8150
+$Comp
+L 74xx:74LS74 U11
+U 2 1 624B3624
+P 7750 8900
+F 0 "U11" H 7550 9150 50  0000 C CNN
+F 1 "74LS74" H 7900 9150 50  0000 C CNN
+F 2 "Package_DIP:DIP-14_W7.62mm_LongPads" H 7750 8900 50  0001 C CNN
+F 3 "74xx/74hc_hct74.pdf" H 7750 8900 50  0001 C CNN
+	2    7750 8900
+	1    0    0    -1
+$EndComp
+Wire Wire Line
+	5400 8750 5400 9350
+Wire Wire Line
+	7750 9350 7750 9200
+Connection ~ 5400 8750
+Wire Wire Line
+	5400 8750 5500 8750
+$Comp
+L power:VCC #PWR?
+U 1 1 624EDA8A
+P 7750 8500
+F 0 "#PWR?" H 7750 8350 50  0001 C CNN
+F 1 "VCC" H 7765 8673 50  0000 C CNN
+F 2 "" H 7750 8500 50  0001 C CNN
+F 3 "" H 7750 8500 50  0001 C CNN
+	1    7750 8500
+	1    0    0    -1
+$EndComp
+Wire Wire Line
+	7750 8600 7750 8500
+Wire Wire Line
+	5400 9350 7300 9350
+Wire Wire Line
+	7450 8800 7300 8800
+Wire Wire Line
+	7300 8800 7300 9350
+Connection ~ 7300 9350
+Wire Wire Line
+	7300 9350 7750 9350
+Text GLabel 7000 8900 0    50   Input ~ 0
+IO_CLOCK
+Wire Wire Line
+	7000 8900 7450 8900
+NoConn ~ 8050 9000
+Wire Wire Line
+	8050 8800 8500 8800
+Text GLabel 8500 8800 2    50   Output ~ 0
+E
 $EndSCHEMATC
