File: CGA_3_6.sch (KiCad schematic (older format))
At the start: 21 parts, among them U1 74S112, U11 74LS74, U12 74LS393, U13 74LS08, U15 74LS00, U16 74LS04, U17 74LS138, U18 74LS138, U19 74LS138, U26 74S04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

Commit message: More sheet 3
Connections:
- net ~Q2': now reaches U4.3 (D0), U42.1, U6.10
Changed lines of the file:
@@
 	1500 1400 1750 1400
 Wire Wire Line
-	5150 2150 5150 3000
+	5150 2150 5150 2650
 $Comp
 L power:VCC #PWR?
@@
 	3200 3800 4200 3800
 Connection ~ 3200 3800
+Text GLabel 5500 2650 2    50   Output ~ 0
+~Q2'
+Wire Wire Line
+	5500 2650 5150 2650
+Connection ~ 5150 2650
+Wire Wire Line
+	5150 2650 5150 3000
 $EndSCHEMATC
