File: CGA_4_6.sch (KiCad schematic (older format))
At the start: 1 part, among them U47 74LS51

Commit message: More sheet 4
Parts:
- added U1: 74S112, Package_DIP:DIP-16_W7.62mm_LongPads, symbol 74xx:74LS112
- added U26: 74S04, Package_DIP:DIP-14_W7.62mm_LongPads, symbol 74xx:74LS04
Connections:
- new net: U1.2 (K), U26.2
- new net 14_MHZ: U1.1 (C)
- new net RAS: U1.3 (J), U26.1
- new net VCC: U1.15 (~R), U1.4 (~S)
Changed lines of the file:
@@
 Text GLabel 850  1700 0    50   Input ~ 0
 ~HRES
+$Comp
+L 74xx:74LS04 U?
+U 1 1 62D1DE1F
+P 1800 2450
+AR Path="/60463C57/62D1DE1F" Ref="U?"  Part="2"
+AR Path="/60463CC5/62D1DE1F" Ref="U26"  Part="1"
+F 0 "U26" H 1750 2150 50  0000 C CNN
+F 1 "74S04" H 1750 2250 50  0000 C CNN
+F 2 "Package_DIP:DIP-14_W7.62mm_LongPads" H 1800 2450 50  0001 C CNN
+F 3 "http://www.ti.com/lit/gpn/sn74LS04" H 1800 2450 50  0001 C CNN
+	1    1800 2450
+	1    0    0    -1
+$EndComp
+$Comp
+L 74xx:74LS112 U1
+U 1 1 62D1E97B
+P 2900 2350
+F 0 "U1" H 2750 2600 50  0000 C CNN
+F 1 "74S112" H 3050 2600 50  0000 C CNN
+F 2 "Package_DIP:DIP-16_W7.62mm_LongPads" H 2900 2350 50  0001 C CNN
+F 3 "http://www.ti.com/lit/gpn/sn74LS112" H 2900 2350 50  0001 C CNN
+	1    2900 2350
+	1    0    0    -1
+$EndComp
+Wire Wire Line
+	2100 2450 2600 2450
+Wire Wire Line
+	1500 2450 1350 2450
+Text GLabel 850  2450 0    50   Input ~ 0
+RAS
+Wire Wire Line
+	1350 2450 1350 2250
+Wire Wire Line
+	1350 2250 2600 2250
+Connection ~ 1350 2450
+Wire Wire Line
+	1350 2450 850  2450
+Text GLabel 1000 2100 0    50   Input ~ 0
+14_MHZ
+Wire Wire Line
+	1000 2100 2200 2100
+Wire Wire Line
+	2200 2100 2200 2350
+Wire Wire Line
+	2200 2350 2600 2350
+Wire Wire Line
+	2900 2650 2900 2750
+Wire Wire Line
+	2900 2750 2450 2750
+Wire Wire Line
+	2450 2750 2450 1950
+Wire Wire Line
+	2450 1950 2900 1950
+Wire Wire Line
+	2900 1950 2900 2050
+$Comp
+L power:VCC #PWR?
+U 1 1 62D5033E
+P 2900 1850
+F 0 "#PWR?" H 2900 1700 50  0001 C CNN
+F 1 "VCC" H 2915 2023 50  0000 C CNN
+F 2 "" H 2900 1850 50  0001 C CNN
+F 3 "" H 2900 1850 50  0001 C CNN
+	1    2900 1850
+	1    0    0    -1
+$EndComp
+Wire Wire Line
+	2900 1950 2900 1850
+Connection ~ 2900 1950
 $EndSCHEMATC

Commit message: More CGA sheet 4
Parts:
- added unit 3 of U26
- added U46: 74LS00, Package_DIP:DIP-14_W7.62mm_LongPads, symbol 74xx:74LS00
Connections:
- net at U47.6: now also U26.5, U46.12, U46.9
- net at U1.5 (Q): now also U46.13, U46.5
- net at U1.6 (~Q): now also U46.10, U46.2
- new net: U26.6, U46.1, U46.4
Other:
- moved on the sheet: U47B
Changed lines of the file:
@@
 L 74xx:74LS51 U47
 U 2 1 62D15655
-P 1850 1400
-F 0 "U47" H 1850 1925 50  0000 C CNN
-F 1 "74LS51" H 1850 1834 50  0000 C CNN
-F 2 "Package_DIP:DIP-14_W7.62mm_LongPads" H 1850 1400 50  0001 C CNN
-F 3 "http://www.ti.com/lit/ds/symlink/sn74ls51.pdf" H 1850 1400 50  0001 C CNN
-	2    1850 1400
-	1    0    0    -1
-$EndComp
+P 1850 1200
+F 0 "U47" H 1850 1725 50  0000 C CNN
+F 1 "74LS51" H 1850 1634 50  0000 C CNN
+F 2 "Package_DIP:DIP-14_W7.62mm_LongPads" H 1850 1200 50  0001 C CNN
+F 3 "http://www.ti.com/lit/ds/symlink/sn74ls51.pdf" H 1850 1200 50  0001 C CNN
+	2    1850 1200
+	1    0    0    -1
+$EndComp
+Wire Wire Line
+	1350 1100 850  1100
+Text GLabel 850  1100 0    50   Input ~ 0
+HRES
 Wire Wire Line
 	1350 1300 850  1300
 Text GLabel 850  1300 0    50   Input ~ 0
-HRES
+Q1
 Wire Wire Line
 	1350 1500 850  1500
 Text GLabel 850  1500 0    50   Input ~ 0
-Q1
-Wire Wire Line
-	1350 1700 850  1700
-Text GLabel 850  1700 0    50   Input ~ 0
 ~HRES
 $Comp
@@
 	2900 1950 2900 1850
 Connection ~ 2900 1950
+$Comp
+L 74xx:74LS04 U?
+U 3 1 62D569A0
+P 2900 1200
+AR Path="/60463C57/62D569A0" Ref="U?"  Part="2"
+AR Path="/60463CC5/62D569A0" Ref="U26"  Part="3"
+F 0 "U26" H 2600 1300 50  0000 C CNN
+F 1 "74S04" H 3100 1300 50  0000 C CNN
+F 2 "Package_DIP:DIP-14_W7.62mm_LongPads" H 2900 1200 50  0001 C CNN
+F 3 "http://www.ti.com/lit/gpn/sn74LS04" H 2900 1200 50  0001 C CNN
+	3    2900 1200
+	1    0    0    -1
+$EndComp
+Wire Wire Line
+	2350 1200 2500 1200
+$Comp
+L 74xx:74LS00 U46
+U 1 1 62D5F730
+P 4000 1400
+F 0 "U46" H 4000 1100 50  0000 C CNN
+F 1 "74LS00" H 4000 1200 50  0000 C CNN
+F 2 "Package_DIP:DIP-14_W7.62mm_LongPads" H 4000 1400 50  0001 C CNN
+F 3 "http://www.ti.com/lit/gpn/sn74ls00" H 4000 1400 50  0001 C CNN
+	1    4000 1400
+	1    0    0    -1
+$EndComp
+$Comp
+L 74xx:74LS00 U46
+U 2 1 62D5E238
+P 4000 1000
+F 0 "U46" H 4000 683 50  0000 C CNN
+F 1 "74LS00" H 4000 774 50  0000 C CNN
+F 2 "Package_DIP:DIP-14_W7.62mm_LongPads" H 4000 1000 50  0001 C CNN
+F 3 "http://www.ti.com/lit/gpn/sn74ls00" H 4000 1000 50  0001 C CNN
+	2    4000 1000
+	1    0    0    1
+$EndComp
+Wire Wire Line
+	3700 1100 3600 1100
+Wire Wire Line
+	3600 1100 3600 1200
+Wire Wire Line
+	3600 1300 3700 1300
+Wire Wire Line
+	3600 1200 3200 1200
+Connection ~ 3600 1200
+Wire Wire Line
+	3600 1200 3600 1300
+Wire Wire Line
+	3200 2250 3400 2250
+Wire Wire Line
+	3400 2250 3400 900
+Wire Wire Line
+	3400 900  3700 900
+Wire Wire Line
+	3200 2450 3550 2450
+Wire Wire Line
+	3550 2450 3550 1500
+Wire Wire Line
+	3550 1500 3700 1500
+$Comp
+L 74xx:74LS00 U46
+U 3 1 62D70773
+P 4000 2800
+F 0 "U46" H 4000 3150 50  0000 C CNN
+F 1 "74LS00" H 4000 3050 50  0000 C CNN
+F 2 "Package_DIP:DIP-14_W7.62mm_LongPads" H 4000 2800 50  0001 C CNN
+F 3 "http://www.ti.com/lit/gpn/sn74ls00" H 4000 2800 50  0001 C CNN
+	3    4000 2800
+	1    0    0    1
+$EndComp
+$Comp
+L 74xx:74LS00 U46
+U 4 1 62D6A442
+P 4000 2350
+F 0 "U46" H 4000 2033 50  0000 C CNN
+F 1 "74LS00" H 4000 2124 50  0000 C CNN
+F 2 "Package_DIP:DIP-14_W7.62mm_LongPads" H 4000 2350 50  0001 C CNN
+F 3 "http://www.ti.com/lit/gpn/sn74ls00" H 4000 2350 50  0001 C CNN
+	4    4000 2350
+	1    0    0    1
+$EndComp
+Wire Wire Line
+	3700 2250 3400 2250
+Connection ~ 3400 2250
+Wire Wire Line
+	3550 2450 3550 2700
+Wire Wire Line
+	3550 2700 3700 2700
+Connection ~ 3550 2450
+Wire Wire Line
+	3700 2450 3600 2450
+Wire Wire Line
+	3600 2450 3600 2650
+Wire Wire Line
+	3600 2900 3700 2900
+Wire Wire Line
+	3600 2650 3250 2650
+Wire Wire Line
+	3250 2650 3250 1450
+Wire Wire Line
+	3250 1450 2500 1450
+Wire Wire Line
+	2500 1450 2500 1200
+Connection ~ 3600 2650
+Wire Wire Line
+	3600 2650 3600 2900
+Connection ~ 2500 1200
+Wire Wire Line
+	2500 1200 2600 1200
 $EndSCHEMATC

Commit message: Some more sheet 4
Parts:
- added U2: 74LS74, Package_DIP:DIP-14_W7.62mm_LongPads, symbol 74xx:74LS74
Connections:
- net Q1: now also U2.3 (C)
- net VCC: now also U2.1 (~R)
- net ~EN_CPU_CAS_ADDR: now reaches U46.6
- net ~EN_CPU_RAS_ADDR: now reaches U46.3
- net ~EN_CRT_CAS_ADDR: now reaches U46.11
- net ~EN_CRT_RAS_ADDR: now reaches U46.8
- new net ~CPU_MEM_SEL: U2.2 (D)
Changed lines of the file:
@@
 Wire Wire Line
 	2500 1200 2600 1200
+$Comp
+L 74xx:74LS74 U2
+U 1 1 62D7E32E
+P 2900 3400
+F 0 "U2" H 2750 3650 50  0000 C CNN
+F 1 "74LS74" H 3050 3650 50  0000 C CNN
+F 2 "Package_DIP:DIP-14_W7.62mm_LongPads" H 2900 3400 50  0001 C CNN
+F 3 "74xx/74hc_hct74.pdf" H 2900 3400 50  0001 C CNN
+	1    2900 3400
+	1    0    0    -1
+$EndComp
+Text GLabel 2100 3300 0    50   Input ~ 0
+~CPU_MEM_SEL
+$Comp
+L power:VCC #PWR?
+U 1 1 62D8D7F8
+P 2700 3750
+F 0 "#PWR?" H 2700 3600 50  0001 C CNN
+F 1 "VCC" V 2715 3877 50  0000 L CNN
+F 2 "" H 2700 3750 50  0001 C CNN
+F 3 "" H 2700 3750 50  0001 C CNN
+	1    2700 3750
+	0    -1   -1   0
+$EndComp
+Wire Wire Line
+	2700 3750 2900 3750
+Wire Wire Line
+	2900 3750 2900 3700
+Wire Wire Line
+	2600 3400 2100 3400
+Text GLabel 2100 3400 0    50   Input ~ 0
+Q1
+Wire Wire Line
+	2100 3300 2600 3300
+Wire Wire Line
+	4300 1000 5350 1000
+Text GLabel 5350 1000 2    50   Output ~ 0
+~EN_CPU_CAS_ADDR
+Text GLabel 5350 1150 2    50   Output ~ 0
+~EN_CPU_RAS_ADDR
+Wire Wire Line
+	5350 1150 4450 1150
+Wire Wire Line
+	4450 1150 4450 1400
+Wire Wire Line
+	4450 1400 4300 1400
+Text GLabel 5350 1300 2    50   Output ~ 0
+~EN_CRT_CAS_ADDR
+Text GLabel 5350 1450 2    50   Output ~ 0
+~EN_CRT_RAS_ADDR
+Wire Wire Line
+	5350 1300 4550 1300
+Wire Wire Line
+	4550 1300 4550 2350
+Wire Wire Line
+	4550 2350 4300 2350
+Wire Wire Line
+	5350 1450 4650 1450
+Wire Wire Line
+	4650 1450 4650 2800
+Wire Wire Line
+	4650 2800 4300 2800
 $EndSCHEMATC

Commit message: More sheet 4
Connections:
- net ~RAS: now reaches U1.2 (K), U26.2
Changed lines of the file:
@@
 $EndComp
 Wire Wire Line
-	2100 2450 2600 2450
+	2100 2450 2200 2450
 Wire Wire Line
 	1500 2450 1350 2450
@@
 Wire Wire Line
 	4650 2800 4300 2800
+Wire Wire Line
+	2200 2450 2200 2850
+Wire Wire Line
+	2200 2850 2700 2850
+Connection ~ 2200 2450
+Wire Wire Line
+	2200 2450 2600 2450
+Text GLabel 2700 2850 2    50   Output ~ 0
+~RAS
 $EndSCHEMATC

Commit message: More sheet 4
Parts:
- added U28: 74LS10, Package_DIP:DIP-14_W7.62mm_LongPads, symbol 74xx:74LS10
- added U29: 74S04, Package_DIP:DIP-14_W7.62mm_LongPads, symbol 74xx:74LS04
- added U49: 74LS02, Package_DIP:DIP-14_W7.62mm_LongPads, symbol 74xx:74LS02
Connections:
- net at U47.2: now also U2.6 (~Q), U28.4
- new net: U28.5, U49.4
- new net: U28.3, U29.2
- new net Q5: U49.6
- new net ~MEMW: U29.1
- new net ~Q2': U49.5
- new net ~WE: U28.6
Other:
- moved on the sheet: U2A
Changed lines of the file:
@@
 L 74xx:74LS74 U2
 U 1 1 62D7E32E
-P 2900 3400
-F 0 "U2" H 2750 3650 50  0000 C CNN
-F 1 "74LS74" H 3050 3650 50  0000 C CNN
-F 2 "Package_DIP:DIP-14_W7.62mm_LongPads" H 2900 3400 50  0001 C CNN
-F 3 "74xx/74hc_hct74.pdf" H 2900 3400 50  0001 C CNN
-	1    2900 3400
+P 2300 3850
+F 0 "U2" H 2150 4100 50  0000 C CNN
+F 1 "74LS74" H 2450 4100 50  0000 C CNN
+F 2 "Package_DIP:DIP-14_W7.62mm_LongPads" H 2300 3850 50  0001 C CNN
+F 3 "74xx/74hc_hct74.pdf" H 2300 3850 50  0001 C CNN
+	1    2300 3850
 	1    0    0    -1
 $EndComp
-Text GLabel 2100 3300 0    50   Input ~ 0
+Text GLabel 1500 3750 0    50   Input ~ 0
 ~CPU_MEM_SEL
 $Comp
 L power:VCC #PWR?
 U 1 1 62D8D7F8
-P 2700 3750
-F 0 "#PWR?" H 2700 3600 50  0001 C CNN
-F 1 "VCC" V 2715 3877 50  0000 L CNN
-F 2 "" H 2700 3750 50  0001 C CNN
-F 3 "" H 2700 3750 50  0001 C CNN
-	1    2700 3750
+P 2100 4200
+F 0 "#PWR?" H 2100 4050 50  0001 C CNN
+F 1 "VCC" V 2115 4327 50  0000 L CNN
+F 2 "" H 2100 4200 50  0001 C CNN
+F 3 "" H 2100 4200 50  0001 C CNN
+	1    2100 4200
 	0    -1   -1   0
 $EndComp
 Wire Wire Line
-	2700 3750 2900 3750
+	2100 4200 2300 4200
 Wire Wire Line
-	2900 3750 2900 3700
+	2300 4200 2300 4150
 Wire Wire Line
-	2600 3400 2100 3400
-Text GLabel 2100 3400 0    50   Input ~ 0
+	2000 3850 1500 3850
+Text GLabel 1500 3850 0    50   Input ~ 0
 Q1
 Wire Wire Line
-	2100 3300 2600 3300
+	1500 3750 2000 3750
 Wire Wire Line
 	4300 1000 5350 1000
@@
 Text GLabel 2700 2850 2    50   Output ~ 0
 ~RAS
+$Comp
+L 74xx:74LS02 U49
+U 2 1 62E07279
+P 4400 3800
+F 0 "U49" H 4400 4125 50  0000 C CNN
+F 1 "74LS02" H 4400 4034 50  0000 C CNN
+F 2 "Package_DIP:DIP-14_W7.62mm_LongPads" H 4400 3800 50  0001 C CNN
+F 3 "http://www.ti.com/lit/gpn/sn74ls02" H 4400 3800 50  0001 C CNN
+	2    4400 3800
+	1    0    0    -1
+$EndComp
+Text GLabel 3800 3700 0    50   Input ~ 0
+~Q2'
+Wire Wire Line
+	3800 3700 4100 3700
+Text GLabel 3800 3900 0    50   Input ~ 0
+Q5
+Wire Wire Line
+	3800 3900 4100 3900
+$Comp
+L 74xx:74LS10 U28
+U 2 1 62E3583A
+P 5500 3900
+F 0 "U28" H 5500 3583 50  0000 C CNN
+F 1 "74LS10" H 5500 3674 50  0000 C CNN
+F 2 "Package_DIP:DIP-14_W7.62mm_LongPads" H 5500 3900 50  0001 C CNN
+F 3 "http://www.ti.com/lit/gpn/sn74LS10" H 5500 3900 50  0001 C CNN
+	2    5500 3900
+	1    0    0    1
+$EndComp
+Wire Wire Line
+	4700 3800 5200 3800
+Wire Wire Line
+	2600 3950 2750 3950
+Wire Wire Line
+	3100 3950 3100 4050
+Wire Wire Line
+	3100 4050 4700 4050
+Wire Wire Line
+	4700 4050 4700 3900
+Wire Wire Line
+	4700 3900 5200 3900
+Wire Wire Line
+	2750 3950 2750 4400
+Wire Wire Line
+	2750 4400 550  4400
+Wire Wire Line
+	550  4400 550  900
+Wire Wire Line
+	550  900  1350 900
+Connection ~ 2750 3950
+Wire Wire Line
+	2750 3950 3100 3950
+$Comp
+L 74xx:74LS04 U?
+U 1 1 62E66435
+P 4300 4450
+AR Path="/60463C57/62E66435" Ref="U?"  Part="2"
+AR Path="/60463CC5/62E66435" Ref="U29"  Part="1"
+F 0 "U29" H 4250 4150 50  0000 C CNN
+F 1 "74S04" H 4250 4250 50  0000 C CNN
+F 2 "Package_DIP:DIP-14_W7.62mm_LongPads" H 4300 4450 50  0001 C CNN
+F 3 "http://www.ti.com/lit/gpn/sn74LS04" H 4300 4450 50  0001 C CNN
+	1    4300 4450
+	1    0    0    -1
+$EndComp
+Wire Wire Line
+	5200 4000 4800 4000
+Wire Wire Line
+	4800 4000 4800 4450
+Wire Wire Line
+	4800 4450 4600 4450
+Text GLabel 3800 4450 0    50   Input ~ 0
+~MEMW
+Wire Wire Line
+	3800 4450 4000 4450
+Text GLabel 6100 3900 2    50   Output ~ 0
+~WE
+Wire Wire Line
+	5800 3900 6100 3900
 $EndSCHEMATC

Commit message: More sheet 4
Parts:
- added unit 2 of U2
- added unit 3 of U29
Connections:
- net ~CPU_MEM_SEL: now also U29.5
- net ~RAS: now also U2.11 (C)
- net at U2.4 (~S): now also U2.13 (~R), U2.9 (Q)
- net at U2.5 (Q): now also U2.12 (D)
- new net: U2.10 (~S), U29.6
- new net XACK: U2.8 (~Q)
Changed lines of the file:
@@
 Q1
 Wire Wire Line
-	1500 3750 2000 3750
+	1500 3750 1700 3750
 Wire Wire Line
 	4300 1000 5350 1000
@@
 Wire Wire Line
 	5800 3900 6100 3900
+$Comp
+L 74xx:74LS74 U2
+U 2 1 62E7CF2E
+P 3350 5350
+F 0 "U2" H 3200 5600 50  0000 C CNN
+F 1 "74LS74" H 3500 5600 50  0000 C CNN
+F 2 "Package_DIP:DIP-14_W7.62mm_LongPads" H 3350 5350 50  0001 C CNN
+F 3 "74xx/74hc_hct74.pdf" H 3350 5350 50  0001 C CNN
+	2    3350 5350
+	1    0    0    -1
+$EndComp
+Wire Wire Line
+	2600 3750 2900 3750
+Wire Wire Line
+	2900 3750 2900 5250
+Wire Wire Line
+	2900 5250 3050 5250
+Wire Wire Line
+	3650 5250 3900 5250
+Wire Wire Line
+	3900 5250 3900 4750
+Wire Wire Line
+	3900 4750 3200 4750
+Wire Wire Line
+	2750 4750 2750 5750
+Wire Wire Line
+	2750 5750 3350 5750
+Wire Wire Line
+	3350 5750 3350 5650
+Wire Wire Line
+	2300 3550 2300 3300
+Wire Wire Line
+	2300 3300 3200 3300
+Wire Wire Line
+	3200 3300 3200 4750
+Connection ~ 3200 4750
+Wire Wire Line
+	3200 4750 2750 4750
+$Comp
+L 74xx:74LS04 U?
+U 3 1 62E96DA9
+P 2150 4900
+AR Path="/60463C57/62E96DA9" Ref="U?"  Part="2"
+AR Path="/60463CC5/62E96DA9" Ref="U29"  Part="3"
+F 0 "U29" H 2100 4600 50  0000 C CNN
+F 1 "74S04" H 2100 4700 50  0000 C CNN
+F 2 "Package_DIP:DIP-14_W7.62mm_LongPads" H 2150 4900 50  0001 C CNN
+F 3 "http://www.ti.com/lit/gpn/sn74LS04" H 2150 4900 50  0001 C CNN
+	3    2150 4900
+	1    0    0    -1
+$EndComp
+Wire Wire Line
+	2450 4900 3350 4900
+Wire Wire Line
+	3350 4900 3350 5050
+Wire Wire Line
+	1700 3750 1700 4900
+Wire Wire Line
+	1700 4900 1850 4900
+Connection ~ 1700 3750
+Wire Wire Line
+	1700 3750 2000 3750
+Text GLabel 2600 5350 0    50   Input ~ 0
+~RAS
+Wire Wire Line
+	2600 5350 3050 5350
+Wire Wire Line
+	3650 5450 4000 5450
+Wire Wire Line
+	4000 5450 4000 4850
+Wire Wire Line
+	4000 4850 5450 4850
+Text GLabel 5450 4850 2    50   Output ~ 0
+XACK
 $EndSCHEMATC

Commit message: more sheet 4
Parts:
- added U62: 74LS125, Package_DIP:DIP-14_W7.62mm_LongPads, symbol 74xx:74LS125
Connections:
- net XACK: now also U62.5
- net ~CPU_MEM_SEL: now also U62.4
- new net IO_READY: U62.6
Changed lines of the file:
@@
 	3650 5450 4000 5450
 Wire Wire Line
-	4000 5450 4000 4850
+	4000 5450 4000 5250
 Wire Wire Line
 	4000 4850 5450 4850
 Text GLabel 5450 4850 2    50   Output ~ 0
 XACK
+$Comp
+L 74xx:74LS125 U62
+U 2 1 62EB767B
+P 4800 5250
+F 0 "U62" H 4800 5567 50  0000 C CNN
+F 1 "74LS125" H 4800 5476 50  0000 C CNN
+F 2 "Package_DIP:DIP-14_W7.62mm_LongPads" H 4800 5250 50  0001 C CNN
+F 3 "http://www.ti.com/lit/gpn/sn74LS125" H 4800 5250 50  0001 C CNN
+	2    4800 5250
+	1    0    0    -1
+$EndComp
+Wire Wire Line
+	4500 5250 4000 5250
+Connection ~ 4000 5250
+Wire Wire Line
+	4000 5250 4000 4850
+Text GLabel 5450 5250 2    50   Output ~ 0
+IO_READY
+Wire Wire Line
+	5450 5250 5100 5250
+Text GLabel 4250 5600 0    50   Input ~ 0
+~CPU_MEM_SEL
+Wire Wire Line
+	4800 5500 4800 5600
+Wire Wire Line
+	4800 5600 4250 5600
 $EndSCHEMATC

Commit message: More sheet 4
Parts:
- added U25: 74LS00, Package_DIP:DIP-14_W7.62mm_LongPads, symbol 74xx:74LS00
- added U30: 74LS32, Package_DIP:DIP-14_W7.62mm_LongPads, symbol 74xx:74LS32
- added unit 1 of U47
Connections:
- net HRES: now also U30.5
- net VCC: now also U47.10, U47.13
- net ~Q2': now also U47.12
- new net: U25.9, U30.6
- new net AT_LATCH: U47.8
- new net CAS_CC: U25.10
- new net CC_LATCH: U25.8
- new net GRPH: U47.1
- new net ~CCLK: U30.4, U47.11
- new net ~GRPH: U47.9
Changed lines of the file:
@@
 Wire Wire Line
 	4800 5600 4250 5600
+$Comp
+L 74xx:74LS32 U?
+U 2 1 62ED8784
+P 5800 3000
+AR Path="/60463C57/62ED8784" Ref="U?"  Part="3"
+AR Path="/60463CC5/62ED8784" Ref="U30"  Part="2"
+F 0 "U30" H 5800 2683 50  0000 C CNN
+F 1 "74LS32" H 5800 2774 50  0000 C CNN
+F 2 "Package_DIP:DIP-14_W7.62mm_LongPads" H 5800 3000 50  0001 C CNN
+F 3 "http://www.ti.com/lit/gpn/sn74LS32" H 5800 3000 50  0001 C CNN
+	2    5800 3000
+	1    0    0    1
+$EndComp
+Text GLabel 5200 2900 0    50   Input ~ 0
+HRES
+Wire Wire Line
+	5200 2900 5500 2900
+Text GLabel 5200 3100 0    50   Input ~ 0
+~CCLK
+Wire Wire Line
+	5500 3100 5400 3100
+$Comp
+L 74xx:74LS00 U25
+U 3 1 62EFF4A5
+P 6650 3100
+F 0 "U25" H 6650 2800 50  0000 C CNN
+F 1 "74LS00" H 6650 2900 50  0000 C CNN
+F 2 "Package_DIP:DIP-14_W7.62mm_LongPads" H 6650 3100 50  0001 C CNN
+F 3 "http://www.ti.com/lit/gpn/sn74ls00" H 6650 3100 50  0001 C CNN
+	3    6650 3100
+	1    0    0    -1
+$EndComp
+Wire Wire Line
+	6350 3000 6100 3000
+Wire Wire Line
+	6350 3200 6100 3200
+Wire Wire Line
+	6100 3200 6100 3300
+Wire Wire Line
+	6100 3300 5200 3300
+Text GLabel 5200 3300 0    50   Input ~ 0
+CAS_CC
+Wire Wire Line
+	6950 3100 7350 3100
+Text GLabel 7350 3100 2    50   Output ~ 0
+CC_LATCH
+$Comp
+L 74xx:74LS51 U47
+U 1 1 62F37BE3
+P 6300 2100
+F 0 "U47" H 6300 2625 50  0000 C CNN
+F 1 "74LS51" H 6300 2534 50  0000 C CNN
+F 2 "Package_DIP:DIP-14_W7.62mm_LongPads" H 6300 2100 50  0001 C CNN
+F 3 "http://www.ti.com/lit/ds/symlink/sn74ls51.pdf" H 6300 2100 50  0001 C CNN
+	1    6300 2100
+	1    0    0    -1
+$EndComp
+Wire Wire Line
+	6800 2100 7200 2100
+Text GLabel 7200 2100 2    50   Output ~ 0
+AT_LATCH
+$Comp
+L power:VCC #PWR?
+U 1 1 62F71B77
+P 5650 1750
+F 0 "#PWR?" H 5650 1600 50  0001 C CNN
+F 1 "VCC" H 5750 1800 50  0000 C CNN
+F 2 "" H 5650 1750 50  0001 C CNN
+F 3 "" H 5650 1750 50  0001 C CNN
+	1    5650 1750
+	1    0    0    -1
+$EndComp
+Text GLabel 5500 1900 0    50   Input ~ 0
+~Q2'
+Wire Wire Line
+	5500 1900 5800 1900
+Wire Wire Line
+	5800 2300 5650 2300
+Wire Wire Line
+	5650 2300 5650 2000
+Wire Wire Line
+	5650 2000 5800 2000
+Wire Wire Line
+	5650 2000 5650 1750
+Connection ~ 5650 2000
+Wire Wire Line
+	5800 2400 5400 2400
+Wire Wire Line
+	5400 2400 5400 3100
+Connection ~ 5400 3100
+Wire Wire Line
+	5400 3100 5200 3100
+Text GLabel 5500 1800 0    50   Input ~ 0
+GRPH
+Wire Wire Line
+	5500 1800 5800 1800
+Text GLabel 5500 2200 0    50   Input ~ 0
+~GRPH
+Wire Wire Line
+	5500 2200 5800 2200
 $EndSCHEMATC
