File: ISA_CGA.kicad_pcb (KiCad board)
At the start: 2 copper layers, 168 parts, among them J1 VIDEO JACK, J2 RGBI Output, P1 1X4 BERG, P2 1X6 BERG, P5 Bus_ISA_8bit, Q1 2N3904, U1 74S112, U10 74153, U101 74S174, U11 74LS74, U12 74LS393, U13 74LS08, U14 74S32, U15 74LS00, U16 74LS04, U17 74LS138, U18 74LS138, U19 74LS138, U2 74LS74, U20 74LS04, U21 74LS174, U22 74LS51, U23 74LS32, U24 74LS244, U25 74LS00, U26 74S04, U27 74LS51, U28 74LS10, U29 74S04, U3 74S86, U30 74LS32, U31 74S08, U32 74LS166, U33 27C256, U34 74LS273, U35 74LS273, U36 74LS244, U37 74LS374, U38 MC6845, U39 74LS174, U4 74S174, U40 74LS174, U41 74LS08, U42 74LS86, U43 74S74, U44 74S74, U45 74LS151, U46 74LS00, U47 74LS51, U48 74LS51, U49 74LS02, U5 74S174, U50 2118, U51 2118, U52 2118, U53 2118, U54 2118, U55 2118, U56 2118, U57 2118, U58 74LS374, U59 74LS374, U6 74LS04, U60 74LS374, U61 74LS374, U62 74LS125, U63 74LS175, U64 74LS164, U65 74LS02, U66 74LS245, U67 74LS244, U68 74LS86, U7 74LS166, U8 74LS166, U9 74153

Commit message: Place some more ICs
Parts:
- moved U65 423.1 mm to (330.8, 188.6)
- moved C68 373.8 mm to (290.2, 184.8)
- moved U62 365.3 mm to (288.9, 188.6)
- moved C67 363.0 mm to (304.2, 184.8)
- moved C65 352.4 mm to (332.1, 184.8)
- moved C66 350.0 mm to (318.1, 184.8)
- moved C64 341.6 mm to (346.1, 184.8)
- moved U66 288.3 mm to (344.8, 188.6)
- moved U64 286.6 mm to (316.9, 188.6)
- moved U63 286.5 mm to (302.9, 188.6)
Changed lines of the file:
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@@
   )
   (module Capacitor_THT:C_Disc_D4.3mm_W1.9mm_P5.00mm (layer F.Cu)
-    (at 368.112 -180.848)
+    (at 290.195 184.785)
     (descr "C, Disc series, Radial, pin pitch=5.00mm, , diameter*width=4.3*1.9mm^2, Capacitor, http://www.vishay.com/docs/45233/krseries.pdf")
     (tags "C Disc series Radial pin pitch 5.00mm  diameter 4.3mm width 1.9mm Capacitor")
-    (fp_text reference C68 (at 2.5 -2.2) (layer F.SilkS)
+    (fp_text reference C68 (at -3.175 0) (layer F.SilkS)
       (effects (font (size 1 1) (thickness 0.15)))
     )
@@
   )
   (module Capacitor_THT:C_Disc_D4.3mm_W1.9mm_P5.00mm (layer F.Cu)
-    (at 359.962 -173.948)
+    (at 304.165 184.785)
     (descr "C, Disc series, Radial, pin pitch=5.00mm, , diameter*width=4.3*1.9mm^2, Capacitor, http://www.vishay.com/docs/45233/krseries.pdf")
     (tags "C Disc series Radial pin pitch 5.00mm  diameter 4.3mm width 1.9mm Capacitor")
-    (fp_text reference C67 (at 2.5 -2.2) (layer F.SilkS)
+    (fp_text reference C67 (at -3.175 0) (layer F.SilkS)
       (effects (font (size 1 1) (thickness 0.15)))
     )
@@
   )
   (module Capacitor_THT:C_Disc_D4.3mm_W1.9mm_P5.00mm (layer F.Cu)
-    (at 351.812 -163.598)
+    (at 318.135 184.785)
     (descr "C, Disc series, Radial, pin pitch=5.00mm, , diameter*width=4.3*1.9mm^2, Capacitor, http://www.vishay.com/docs/45233/krseries.pdf")
     (tags "C Disc series Radial pin pitch 5.00mm  diameter 4.3mm width 1.9mm Capacitor")
-    (fp_text reference C66 (at 2.5 -2.2) (layer F.SilkS)
+    (fp_text reference C66 (at -3.175 0) (layer F.SilkS)
       (effects (font (size 1 1) (thickness 0.15)))
     )
@@
   )
   (module Capacitor_THT:C_Disc_D4.3mm_W1.9mm_P5.00mm (layer F.Cu)
-    (at 351.812 -167.048)
+    (at 332.105 184.785)
     (descr "C, Disc series, Radial, pin pitch=5.00mm, , diameter*width=4.3*1.9mm^2, Capacitor, http://www.vishay.com/docs/45233/krseries.pdf")
     (tags "C Disc series Radial pin pitch 5.00mm  diameter 4.3mm width 1.9mm Capacitor")
-    (fp_text reference C65 (at 2.5 -2.2) (layer F.SilkS)
+    (fp_text reference C65 (at -3.175 0) (layer F.SilkS)
       (effects (font (size 1 1) (thickness 0.15)))
     )
@@
   )
   (module Capacitor_THT:C_Disc_D4.3mm_W1.9mm_P5.00mm (layer F.Cu)
-    (at 335.512 -156.698)
+    (at 346.075 184.785)
     (descr "C, Disc series, Radial, pin pitch=5.00mm, , diameter*width=4.3*1.9mm^2, Capacitor, http://www.vishay.com/docs/45233/krseries.pdf")
     (tags "C Disc series Radial pin pitch 5.00mm  diameter 4.3mm width 1.9mm Capacitor")
-    (fp_text reference C64 (at 2.5 -2.2) (layer F.SilkS)
+    (fp_text reference C64 (at -3.175 0) (layer F.SilkS)
       (effects (font (size 1 1) (thickness 0.15)))
     )
@@
   )
   (module Package_DIP:DIP-20_W7.62mm_LongPads (layer F.Cu)
-    (at 199.294 -60.232)
+    (at 344.805 188.595)
     (descr "20-lead though-hole mounted DIP package, row spacing 7.62 mm (300 mils), LongPads")
     (tags "THT DIP DIL PDIP 2.54mm 7.62mm 300mil LongPads")
-    (fp_text reference U66 (at 3.81 -2.33) (layer F.SilkS)
+    (fp_text reference U66 (at -2.54 0 90) (layer F.SilkS)
       (effects (font (size 1 1) (thickness 0.15)))
     )
@@
   )
   (module Package_DIP:DIP-14_W7.62mm_LongPads (layer F.Cu)
-    (at 78.844 -151.282)
+    (at 330.835 188.595)
     (descr "14-lead though-hole mounted DIP package, row spacing 7.62 mm (300 mils), LongPads")
     (tags "THT DIP DIL PDIP 2.54mm 7.62mm 300mil LongPads")
-    (fp_text reference U65 (at 3.81 -2.33) (layer F.SilkS)
+    (fp_text reference U65 (at -2.54 0 90) (layer F.SilkS)
       (effects (font (size 1 1) (thickness 0.15)))
     )
@@
   )
   (module Package_DIP:DIP-14_W7.62mm_LongPads (layer F.Cu)
-    (at 305.014 -97.792)
+    (at 316.865 188.595)
     (descr "14-lead though-hole mounted DIP package, row spacing 7.62 mm (300 mils), LongPads")
     (tags "THT DIP DIL PDIP 2.54mm 7.62mm 300mil LongPads")
-    (fp_text reference U64 (at 3.81 -2.33) (layer F.SilkS)
+    (fp_text reference U64 (at -2.54 0 90) (layer F.SilkS)
       (effects (font (size 1 1) (thickness 0.15)))
     )
@@
   )
   (module Package_DIP:DIP-16_W7.62mm_LongPads (layer F.Cu)
-    (at 293.414 -97.792)
+    (at 302.895 188.595)
     (descr "16-lead though-hole mounted DIP package, row spacing 7.62 mm (300 mils), LongPads")
     (tags "THT DIP DIL PDIP 2.54mm 7.62mm 300mil LongPads")
-    (fp_text reference U63 (at 3.81 -2.33) (layer F.SilkS)
+    (fp_text reference U63 (at -2.54 0 90) (layer F.SilkS)
       (effects (font (size 1 1) (thickness 0.15)))
     )
@@
   )
   (module Package_DIP:DIP-14_W7.62mm_LongPads (layer F.Cu)
-    (at 113.644 -131.882)
+    (at 288.925 188.595)
     (descr "14-lead though-hole mounted DIP package, row spacing 7.62 mm (300 mils), LongPads")
     (tags "THT DIP DIL PDIP 2.54mm 7.62mm 300mil LongPads")
-    (fp_text reference U62 (at 3.81 -2.33) (layer F.SilkS)
+    (fp_text reference U62 (at -2.54 0 90) (layer F.SilkS)
       (effects (font (size 1 1) (thickness 0.15)))
     )

Commit message: Place more components
Parts:
- moved C69 422.1 mm to (135.3, 174.6)
- moved C70 403.1 mm to (151.8, 174.6)
- moved C71 381.8 mm to (168.3, 174.6)
- moved C73 379.0 mm to (196.2, 192.4), turned to 90 degrees
- moved C72 376.8 mm to (184.8, 174.6)
- moved U34 346.2 mm to (134.0, 178.4)
- moved U35 344.8 mm to (150.5, 178.4)
- moved U37 339.1 mm to (183.5, 178.4)
- moved U36 335.3 mm to (167.0, 178.4)
- moved U38 298.9 mm to (200.0, 197.5), turned to 90 degrees
- moved U33 1.27 mm to (109.9, 168.3)
- moved C35 1.27 mm to (114.9, 164.3)

Commit message: place all components
Parts:
- moved C80 378.7 mm to (208.3, 179.7)
- moved C79 371.0 mm to (223.5, 174.6)
- moved C75 359.3 mm to (238.8, 174.6)
- moved C78 347.9 mm to (254.0, 174.6)
- moved C77 346.8 mm to (269.2, 174.6)
- moved C74 341.5 mm to (254.0, 148.0)
- moved C76 333.4 mm to (269.2, 148.0)
- moved U101 320.1 mm to (207.0, 183.5)
- moved C44 312.8 mm to (147.3, 99.1)
- moved U61 308.0 mm to (268.0, 178.4)
- moved U39 304.9 mm to (252.7, 151.8)
- moved P5 303.5 mm to (334.6, 207.6)
- moved J2 295.0 mm to (389.1, 155.4), turned to 90 degrees
- moved U60 292.9 mm to (252.7, 178.4)
- moved C26 286.1 mm to (368.9, 197.5)
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Other:
- board outline added: 369.3 x 117.6 mm
- copper layers 2 -> 4
- net class POWER: via_dia 0.8 -> 1.2
