File: CGA_5_6.kicad_sch (KiCad schematic)
At the start: 40 parts, among them Q1 2N3904, U13 74LS08, U14 74S32, U15 74LS00, U21 74LS174, U24 74LS244, U41 74LS08, U43 74S74, U44 74S74, U45 74LS151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

Commit message: Fix Q1' naming thanks to Michael Karcher
Parts:
- gave numbers to parts that had none: 2
Connections:
- net CURSOR: now also U20.1; no longer U20.5
- net DISPEN: now also U20.3; no longer U20.5
- net ~{DISPEN}: now also U20.4; no longer U20.6
- net at U24.2: now also U20.12; no longer U20.6
- net at U21.3 (D0): now also U20.2; no longer U20.6
- net at U64.1 (DSA): now also U42.8; no longer U42.3
- net at U64.12 (Q6): now also U20.11; no longer U20.5
- net at U63.9 (Cp), U64.4 (Q1), U67.11 (I0b): now also U42.5; no longer U42.2
- net at U64.6 (Q3): now also U42.10; no longer U42.2
- net at U15.6: now also U42.9; no longer U42.1
- net at U14.12: now also U20.10; no longer U20.6
- net at U41.8, U67.13 (I1b): now also U42.4; no longer U42.1
- new net: U20.13, U42.6
