File: CGA_6_6.kicad_sch (KiCad schematic)
At the start: 89 parts, among them J1 COMPOSITE OUT, J2 RGBI Output, P1 1X4 BERG, P2 1X6 BERG, P5 Bus_ISA_8bit, U13 74LS08, U14 74S32, U26 74S04, U41 74LS08, U66 74LS245

Commit message: Fix Q1' naming thanks to Michael Karcher
Parts:
- gave numbers to parts that had none: 6
Connections:
- net GND: now also U42.13; no longer U42.2
- net RESET: now also U20.9; no longer U20.5
- net ~{MEMR}: now also U42.11; no longer U42.3
- net ~{RESET'}: now also U20.8; no longer U20.6
- net ~{SMEMR}: now also U42.12; no longer U42.1
